File: board for mt8870/board for mt8870.kicad_sch (KiCad schematic)
At the start: 10 parts, among them IC1 MT8870CE, X1 3.579545M

Commit message: generated gerbers
Parts:
- added C1, C2: 220nF, Capacitor_THT:C_Rect_L7.0mm_W3.5mm_P5.00mm, symbol Device:C
- added D1, D2: DIODE, Diode_THT:D_A-405_P5.08mm_Vertical_AnodeUp, symbol pspice:DIODE
- added J2: 6P4C, Connector_RJ:RJ14_Connfly_DS1133-S4_Horizontal, symbol Connector:6P4C
- added J4: power, Connector_PinHeader_2.54mm:PinHeader_1x02_P2.54mm_Vertical, symbol Connector_Generic:Conn_01x02
- added R1, R4, R5: 100k, Resistor_THT:R_Axial_DIN0207_L6.3mm_D2.5mm_P5.08mm_Vertical, symbol Device:R
- added R2: 60.4k, Resistor_THT:R_Axial_DIN0207_L6.3mm_D2.5mm_P5.08mm_Vertical, symbol Device:R
- added R3: 37.4k, Resistor_THT:R_Axial_DIN0207_L6.3mm_D2.5mm_P5.08mm_Vertical, symbol Device:R
- C3, C4: renamed from C?; footprint (none) -> Capacitor_SMD:C_0603_1608Metric
- C5: renamed from C1; value 0.1iF -> 0.1uF; footprint (none) -> Capacitor_SMD:C_0603_1608Metric
- D3: renamed from D?; footprint (none) -> Diode_THT:D_A-405_P5.08mm_Vertical_AnodeUp
- J1: renamed from J?; footprint (none) -> Connector_PinHeader_2.54mm:PinHeader_1x03_P2.54mm_Vertical
- J3: renamed from J?; footprint (none) -> Connector_PinHeader_2.54mm:PinHeader_1x07_P2.54mm_Vertical
- R6: renamed from R2; footprint (none) -> Resistor_THT:R_Axial_DIN0207_L6.3mm_D2.5mm_P5.08mm_Vertical
- R7: renamed from R1; value R -> 330k; footprint (none) -> Resistor_THT:R_Axial_DIN0207_L6.3mm_D2.5mm_P5.08mm_Vertical
- X1: footprint (none) -> Crystal:Crystal_HC49-U_Vertical
Connections:
- net +5V: now also J4.1 (Pin_1)
- net GND: now also J4.2 (Pin_2)
- net IN+: now reaches IC1.1 (IN+)
- net IN+: now also D1.1 (K), D2.2 (A), R1.1, R3.2
- net IN-: now reaches IC1.2 (IN-)
- net IN-: now also D1.2 (A), D2.1 (K), R2.2, R4.1, R5.1
- net GS: now reaches IC1.3 (GS)
- net GS: now also R5.2
- net Vref: now reaches IC1.4 (VREF)
- net Vref: now also R2.1, R3.1
- new net: C1.1, R1.2
- new net: C1.2, J2.3
- new net: C2.1, R4.2
- new net: C2.2, J2.2
Other:
- note added: "both grounded on ALEPH"
